Commit message: change scaling

File: light_weight/urdf/TOCABI.urdf (robot description, URDF)
Before this commit: robot FullBody_Simplified, 37 links, 36 joints
Links:
- link LL_Ankle_1v4_1: geometry collision mesh filename=package://meshes/LL_Ankle_1v4_1.stl scale=1.0 1.0 1.0; visual mesh filename=package://meshes/LL_Ankle_1v4_1.stl scale=1.0 1.0 1.0
- link LL_Ankle_2v7_1: mass 1.9346899212969202 -> 2.0994891576983727; geometry collision mesh filename=package://meshes/LL_Ankle_2v7_1.stl scale=1.0 1.0 1.0; visual mesh filename=package://meshes/LL_Ankle_2v7_1.stl scale=1.0 1.0 1.0
- link LL_Footv1_1: geometry collision mesh filename=package://meshes/LL_Footv1_1.stl scale=1.0 1.0 1.0; visual mesh filename=package://meshes/LL_Footv1_1.stl scale=1.0 1.0 1.0
- link LL_Hip_1v5_1: geometry collision mesh filename=package://meshes/LL_Hip_1v5_1.stl scale=1.0 1.0 1.0; visual mesh filename=package://meshes/LL_Hip_1v5_1.stl scale=1.0 1.0 1.0
- link LL_Hip_2v4_1: geometry collision mesh filename=package://meshes/LL_Hip_2v4_1.stl scale=1.0 1.0 1.0; visual mesh filename=package://meshes/LL_Hip_2v4_1.stl scale=1.0 1.0 1.0
- link LL_Hip_3v5_1: mass 4.748394171510706 -> 5.64595764653467; geometry collision mesh filename=package://meshes/LL_Hip_3v5_1.stl scale=1.0 1.0 1.0; visual mesh filename=package://meshes/LL_Hip_3v5_1.stl scale=1.0 1.0 1.0
- link LL_Knee_1v4_1: mass 2.1717822655770376 -> 2.6111042033255614; geometry collision mesh filename=package://meshes/LL_Knee_1v4_1.stl scale=1.0 1.0 1.0; visual mesh filename=package://meshes/LL_Knee_1v4_1.stl scale=1.0 1.0 1.0
- link LR_Ankle_1v2_1: geometry collision mesh filename=package://meshes/LR_Ankle_1v2_1.stl scale=1.0 1.0 1.0; visual mesh filename=package://meshes/LR_Ankle_1v2_1.stl scale=1.0 1.0 1.0
- link LR_Ankle_2v3_1: mass 1.924891327220748 -> 2.0896905636222005; geometry collision mesh filename=package://meshes/LR_Ankle_2v3_1.stl scale=1.0 1.0 1.0; visual mesh filename=package://meshes/LR_Ankle_2v3_1.stl scale=1.0 1.0 1.0
- link LR_Footv2_2: geometry collision mesh filename=package://meshes/LR_Footv2_2.stl scale=1.0 1.0 1.0; visual mesh filename=package://meshes/LR_Footv2_2.stl scale=1.0 1.0 1.0
- link LR_Hip_1v2_1: geometry collision mesh filename=package://meshes/LR_Hip_1v2_1.stl scale=1.0 1.0 1.0; visual mesh filename=package://meshes/LR_Hip_1v2_1.stl scale=1.0 1.0 1.0
- link LR_Hip_2v3_1: geometry collision mesh filename=package://meshes/LR_Hip_2v3_1.stl scale=1.0 1.0 1.0; visual mesh filename=package://meshes/LR_Hip_2v3_1.stl scale=1.0 1.0 1.0
- link LR_Hip_3v5_1: mass 4.752611894817338 -> 5.650175369841302; geometry collision mesh filename=package://meshes/LR_Hip_3v5_1.stl scale=1.0 1.0 1.0; visual mesh filename=package://meshes/LR_Hip_3v5_1.stl scale=1.0 1.0 1.0
- link LR_Knee_1v6_1: mass 2.1744274951371314 -> 2.613749432885655; geometry collision mesh filename=package://meshes/LR_Knee_1v6_1.stl scale=1.0 1.0 1.0; visual mesh filename=package://meshes/LR_Knee_1v6_1.stl scale=1.0 1.0 1.0
- link L_Pelvisv15_1: mass 10.036811625847252 -> 12.901786749235924; geometry collision mesh filename=package://meshes/L_Pelvisv15_1.stl scale=1.0 1.0 1.0; visual mesh filename=package://meshes/L_Pelvisv15_1.stl scale=1.0 1.0 1.0
- link UL_Arm_1v1_1: geometry collision mesh filename=package://meshes/UL_Arm_1v1_1.stl scale=1.0 1.0 1.0; visual mesh filename=package://meshes/UL_Arm_1v1_1.stl scale=1.0 1.0 1.0
- link UL_Arm_2v1_1: mass 1.1202659214049093 -> 1.9252498488611527; geometry collision mesh filename=package://meshes/UL_Arm_2v1_1.stl scale=1.0 1.0 1.0; visual mesh filename=package://meshes/UL_Arm_2v1_1.stl scale=1.0 1.0 1.0
- link UL_Arm_3v1_1: geometry collision mesh filename=package://meshes/UL_Arm_3v1_1.stl scale=1.0 1.0 1.0; visual mesh filename=package://meshes/UL_Arm_3v1_1.stl scale=1.0 1.0 1.0
- link UL_Shoulder_1v3_1: mass 0.4784016701329476 -> 1.6149801443567293; geometry collision mesh filename=package://meshes/UL_Shoulder_1v3_1.stl scale=1.0 1.0 1.0; visual mesh filename=package://meshes/UL_Shoulder_1v3_1.stl scale=1.0 1.0 1.0
- link UL_Shoulder_2v3_1: geometry collision mesh filename=package://meshes/UL_Shoulder_2v3_1.stl scale=1.0 1.0 1.0; visual mesh filename=package://meshes/UL_Shoulder_2v3_1.stl scale=1.0 1.0 1.0
- link UL_Shoulder_3v3_1: mass 1.6983659250719216 -> 2.834944399295703; geometry collision mesh filename=package://meshes/UL_Shoulder_3v3_1.stl scale=1.0 1.0 1.0; visual mesh filename=package://meshes/UL_Shoulder_3v3_1.stl scale=1.0 1.0 1.0
- link UL_Wrist_1v1_1: mass 0.49848861390960736 -> 0.7829866998307424; geometry collision mesh filename=package://meshes/UL_Wrist_1v1_1.stl scale=1.0 1.0 1.0; visual mesh filename=package://meshes/UL_Wrist_1v1_1.stl scale=1.0 1.0 1.0
- link UL_Wrist_2v1_1: geometry collision mesh filename=package://meshes/UL_Wrist_2v1_1.stl scale=1.0 1.0 1.0; visual mesh filename=package://meshes/UL_Wrist_2v1_1.stl scale=1.0 1.0 1.0
- link UR_Arm_1v2_1: geometry collision mesh filename=package://meshes/UR_Arm_1v2_1.stl scale=1.0 1.0 1.0; visual mesh filename=package://meshes/UR_Arm_1v2_1.stl scale=1.0 1.0 1.0
- link UR_Arm_2v6_1: mass 0.3152819939464439 -> 1.925249848858931; geometry collision mesh filename=package://meshes/UR_Arm_2v6_1.stl scale=1.0 1.0 1.0; visual mesh filename=package://meshes/UR_Arm_2v6_1.stl scale=1.0 1.0 1.0
- link UR_Arm_3v3_1: geometry collision mesh filename=package://meshes/UR_Arm_3v3_1.stl scale=1.0 1.0 1.0; visual mesh filename=package://meshes/UR_Arm_3v3_1.stl scale=1.0 1.0 1.0
- link UR_Hand_1v3_1: mass 0.23815245620329029 -> 0.3159262316423516; geometry collision mesh filename=package://meshes/UR_Hand_1v3_1.stl scale=1.0 1.0 1.0; visual mesh filename=package://meshes/UR_Hand_1v3_1.stl scale=1.0 1.0 1.0
- link UR_Shoulder_1v3_1: mass 0.47840167013294754 -> 1.6149801443567293; geometry collision mesh filename=package://meshes/UR_Shoulder_1v3_1.stl scale=1.0 1.0 1.0; visual mesh filename=package://meshes/UR_Shoulder_1v3_1.stl scale=1.0 1.0 1.0
- link UR_Shoulder_2v2_1: geometry collision mesh filename=package://meshes/UR_Shoulder_2v2_1.stl scale=1.0 1.0 1.0; visual mesh filename=package://meshes/UR_Shoulder_2v2_1.stl scale=1.0 1.0 1.0
- link UR_Shoulder_3v2_1: mass 0.56178745084814 -> 2.834944399295703; geometry collision mesh filename=package://meshes/UR_Shoulder_3v2_1.stl scale=1.0 1.0 1.0; visual mesh filename=package://meshes/UR_Shoulder_3v2_1.stl scale=1.0 1.0 1.0
- link UR_Wrist_1v6_1: mass 0.4704162631935058 -> 0.7829866998307424; geometry collision mesh filename=package://meshes/UR_Wrist_1v6_1.stl scale=1.0 1.0 1.0; visual mesh filename=package://meshes/UR_Wrist_1v6_1.stl scale=1.0 1.0 1.0
- link UR_Wrist_2v3_1: geometry collision mesh filename=package://meshes/UR_Wrist_2v3_1.stl scale=1.0 1.0 1.0; visual mesh filename=package://meshes/UR_Wrist_2v3_1.stl scale=1.0 1.0 1.0
- link U_Body_1v21_1: mass 13.434139763717132 -> 20.03358554636745; geometry collision mesh filename=package://meshes/U_Body_1v21_1.stl scale=1.0 1.0 1.0; visual mesh filename=package://meshes/U_Body_1v21_1.stl scale=1.0 1.0 1.0
- link U_Neck_1v4_1: mass 0.28464806125456393 -> 0.40364564128614283; geometry collision mesh filename=package://meshes/U_Neck_1v4_1.stl scale=1.0 1.0 1.0; visual mesh filename=package://meshes/U_Neck_1v4_1.stl scale=1.0 1.0 1.0
- link U_Neck_2_simv5_1: geometry collision mesh filename=package://meshes/U_Neck_2_simv5_1.stl scale=1.0 1.0 1.0; visual mesh filename=package://meshes/U_Neck_2_simv5_1.stl scale=1.0 1.0 1.0
- link U_Waist_1v3_1: mass 2.69908052620212 -> 3.8814634771227143; geometry collision mesh filename=package://meshes/U_Waist_1v3_1.stl scale=1.0 1.0 1.0; visual mesh filename=package://meshes/U_Waist_1v3_1.stl scale=1.0 1.0 1.0
- link U_Waist_2v8_1: geometry collision mesh filename=package://meshes/U_Waist_2v8_1.stl scale=1.0 1.0 1.0; visual mesh filename=package://meshes/U_Waist_2v8_1.stl scale=1.0 1.0 1.0
Joints:
- joint Revolute100: axis -8.753459365229917e-15 -1.0000000000000007 5.797004494381741e-15 -> -8.753459365229937e-15 2.0227461892159993e-14 1.0000000000000007; origin xyz=0.11000000000058999 0.8108999999999992 0.08480049999999428 rpy=0 0 0 -> xyz=0.11000000000059132 -0.10019949999999271 0.9391000000000024 rpy=0 0 0
- joint Revolute101: axis -1.0 9.658055218388878e-15 8.058026186910817e-15 -> -0.9999999999999997 7.225358918441806e-15 -9.658055218389e-15; origin xyz=-0.05199999999999929 0.08500000000000041 -1.3877787807814457e-16 rpy=0 0 0 -> xyz=-0.051999999999999366 -2.0250467969162858e-15 -0.085 rpy=0 0 0
- joint Revolute102: axis -7.969038271337877e-15 -5.7232163070896695e-15 -1.0 -> -7.136371002869012e-15 -0.9999999999999997 2.0154017343898583e-14; origin xyz=-1.2649568694081403e-05 0.34999999979266283 -1.915134717478395e-15 rpy=0 0 0 -> xyz=-1.2649568694094172e-05 -6.8389738316909644e-15 -0.34999999979266294 rpy=0 0 0
- joint Revolute103: axis 8.35761632995666e-15 6.652281957493676e-15 0.9999999999999962 -> 7.524949061487823e-15 0.9999999999999962 -2.1083600012600796e-14; origin xyz=3.372302437298913e-15 0.3499999999999963 -6.2727600891321345e-15 rpy=0 0 0 -> xyz=3.375077994860476e-15 -1.1803891197814665e-14 -0.34999999999999504 rpy=0 0 0
- joint Revolute104: axis 6.655151913143603e-15 -1.482417119359301e-14 0.9999999999999998 -> 5.822484644674764e-15 0.9999999999999996 3.9291486730870894e-16; origin xyz=-1.204713983096739e-05 0.34999999979266383 -5.079270337660091e-15 rpy=0 0 0 -> xyz=-1.2047139830926313e-05 -9.086065233532282e-15 -0.34999999979266405 rpy=0 0 0
- joint Revolute105: axis -1.0 1.086147058441e-14 6.682907488759382e-15 -> -0.9999999999999997 5.850240220290362e-15 -1.0861470584410102e-14; origin xyz=-0.05549999999999965 6.661338147750939e-16 0.04400000000000051 rpy=0 0 0 -> xyz=-0.05549999999999959 0.04399999999999988 -1.8474111129762605e-15 rpy=0 0 0
- joint Revolute106: axis -1.0 9.569493538878896e-15 8.385371905572258e-15 -> -0.9999999999999997 7.552704637103256e-15 -9.569493538879027e-15; origin xyz=-0.055500000000000285 2.220446049250313e-16 -0.04399999999999972 rpy=0 0 0 -> xyz=-0.055500000000000285 -0.0440000000000001 -3.552713678800501e-16 rpy=0 0 0
- joint Revolute107: axis 1.905207805926619e-14 0.018783332176703096 -0.9998235776537487 -> 1.9735531699801058e-14 -1.000000000000001 1.7420093145759097e-14; origin xyz=-1.1102230246251565e-15 -0.028199523342105376 0.036976842527156134 rpy=0 0 0 -> xyz=-1.092459456231154e-15 0.03749999999999897 0.027500000000001138 rpy=0 0 0
- joint Revolute114: axis 3.0730666689294478e-15 -0.9998235776537486 -0.01878333217670054 -> 3.0461818205712783e-15 1.999442278410868e-14 1.000000000000001; origin xyz=-0.0373000000000015 0.12807740029744474 0.002406144851834713 rpy=0 0 0 -> xyz=-0.03730000000000144 -3.126388037344441e-15 -0.12809999999999974 rpy=0 0 0
- joint Revolute116: axis -5.7220983182086546e-15 -0.9165284694878766 -0.3999694546064873 -> -2.417068170382385e-15 0.008726535498401798 0.9999619230641716; origin xyz=-0.029699999999999227 0.10156705141127464 0.07978335708416867 rpy=0 0 0 -> xyz=-0.0296999999999999 0.03140794556228734 -0.12527885278672074 rpy=0 0 0
- joint Revolute118: axis 0.9999999999999998 -1.934870727800474e-14 3.012787411269809e-14 -> 0.9999999999999996 3.6607934209678794e-14 2.058999505931722e-15; origin xyz=0.03699999947547994 0.13179679391235588 0.05751560757241336 rpy=0 0 0 -> xyz=0.03699999947547971 -0.0012548758046695596 -0.14379452453662794 rpy=0 0 0
- joint Revolute119: axis 3.6365077198379e-14 0.415100422380136 -0.9097755983427095 -> 3.753430374577826e-14 -0.999999628736703 -0.0008616997498676732; origin xyz=-0.02950000000001085 0.05882039413732809 -0.013281989065275335 rpy=0 0 0 -> xyz=-0.029500000000010813 -0.03645862486090994 -0.048031434220230554 rpy=0 0 0
- joint Revolute120: axis -1.0 -3.056184286371969e-15 6.0440899793445875e-15 -> -0.9999999999999997 5.416975350918763e-15 2.915232109023415e-15; origin xyz=0.030999999999999195 0.2075739388700688 -0.02860611651316991 rpy=0 0 0 -> xyz=0.03099999999999918 -0.03250000000000412 -0.20699999999999905 rpy=0 0 0
- joint Revolute48: axis 8.135850272080543e-15 1.0000000000000007 -5.881300216741402e-15 -> 8.135850272080565e-15 -2.0311009818474446e-14 -1.0000000000000007; origin xyz=0.11000000000058976 0.6805999999999996 0.18730049999999515 rpy=0 0 0 -> xyz=0.11000000000059089 0.002300500000009677 1.0694000000000008 rpy=0 0 0
- joint Revolute49: axis 1.4360629127321063e-15 -5.873644089593395e-15 -1.0000000000000002 -> 2.2687301812009516e-15 -0.9999999999999998 2.0304938286308574e-14; origin xyz=-8.881784197001252e-16 -0.08499999999999974 0.0540000000000006 rpy=0 0 0 -> xyz=-9.059419880941278e-16 0.05400000000000227 0.084999999999999 rpy=0 0 0
- joint Revolute51: axis 1.0000000000000004 -7.95667976999021e-15 1.356581037105798e-15 -> 0.9999999999999999 2.1892483055747788e-15 7.956679769990199e-15; origin xyz=-0.06599999999999992 0.0 -0.05400000000000002 rpy=0 0 0 -> xyz=-0.06599999999999988 -0.05400000000000014 2.842170943040401e-16 rpy=0 0 0
- joint Revolute53: axis 2.800832321714712e-15 0.9998235776537475 0.018783332176700362 -> 2.827717170072879e-15 -2.0147078449994638e-14 -1.0; origin xyz=0.08900000000035965 -0.22456723076101626 -0.15824603902887713 rpy=0 0 0 -> xyz=0.08900000000035978 -0.15399999999999658 0.22750000000000511 rpy=0 0 0
- joint Revolute54: axis -2.05230925903742e-14 -0.01878333217670006 0.9998235776537472 -> -2.1206546230909074e-14 0.9999999999999996 -2.0424634206150927e-14; origin xyz=1.3877787807814457e-16 -0.06434802092026792 -0.03531490058947827 rpy=0 0 0 -> xyz=3.552713678800501e-17 -0.03409999999999945 0.06499999999999971 rpy=0 0 0
- joint Revolute55: axis 0.9999999999999998 -3.3977472609707566e-15 2.0426723347466497e-14 -> 0.9999999999999996 2.1170394272997545e-14 3.0403507408677246e-15; origin xyz=0.032900000000002316 0.0021600832003204617 -0.11497971143018008 rpy=0 0 0 -> xyz=0.03290000000000236 -0.11499999999999976 1.7053025658242404e-15 rpy=0 0 0
- joint Revolute58: axis 2.7611417940639986e-15 0.9998235776537469 0.018783332176698638 -> 2.788026642422156e-15 -2.1860985244259824e-14 -0.9999999999999994; origin xyz=-0.03099999999999903 0.12558840550246153 -0.030146349751659668 rpy=0 0 0 -> xyz=-0.030999999999998983 -0.03250000000000369 -0.12499999999999901 rpy=0 0 0
- joint Revolute72: axis -2.7602297695390973e-15 -0.9998235776537489 -0.018783332176704155 -> -2.787114617897265e-15 1.6382728507124966e-14 1.0000000000000016; origin xyz=0.030000000000356117 -0.3794330477195974 -0.007128274561058218 rpy=0 0 0 -> xyz=0.030000000000356124 6.906142324680786e-15 0.3794999999999999 rpy=0 0 0
- joint Revolute74: axis -7.546779104011158e-15 -1.0000000000000007 5.797004494381731e-15 -> -7.546779104011179e-15 2.0227461892159993e-14 1.0000000000000007; origin xyz=0.11000000000059164 0.8109000000000003 0.28980049999999435 rpy=0 0 0 -> xyz=0.11000000000059271 0.10480050000000717 0.9390999999999983 rpy=0 0 0
- joint Revolute76: axis -1.0 7.0862724607023404e-15 8.058026186910835e-15 -> -0.9999999999999997 7.225358918441863e-15 -7.0862724607024596e-15; origin xyz=-0.05199999999999958 0.0850000000000003 -1.1102230246251565e-16 rpy=0 0 0 -> xyz=-0.05199999999999955 -2.078337502098293e-15 -0.085 rpy=0 0 0
- joint Revolute77: axis 8.030270611295247e-15 5.79006560047776e-15 1.0 -> 7.197603342826392e-15 0.9999999999999997 -2.022080419772369e-14; origin xyz=0.05199999999999972 -5.551115123125783e-16 -0.04400000000000043 rpy=0 0 0 -> xyz=0.05199999999999966 -0.044000000000000455 9.947598300641404e-16 rpy=0 0 0
- joint Revolute79: axis 6.6551519131435955e-15 -1.4824171193592992e-14 0.9999999999999984 -> 5.822484644674758e-15 0.9999999999999984 3.9268575288735353e-16; origin xyz=3.6637359812630166e-15 0.3499999999999992 6.494804694057166e-15 rpy=0 0 0 -> xyz=3.588240815588506e-15 4.440892098500626e-16 -0.34999999999999853 rpy=0 0 0
- joint Revolute83: axis -8.030270611295248e-15 -5.912530280392494e-15 -1.0 -> -7.197603342826392e-15 -0.9999999999999997 2.0343102202780055e-14; origin xyz=0.05200000000000037 -1.1102230246251565e-16 0.043999999999999595 rpy=0 0 0 -> xyz=0.05200000000000038 0.04400000000000038 -9.947598300641404e-16 rpy=0 0 0
- joint Revolute87: axis 2.774592544632578e-15 0.9998235776537481 0.018783332176700435 -> 2.8014773929907452e-15 -2.0085214567129895e-14 -1.0000000000000007; origin xyz=0.08900000000035366 -0.23035249707144007 0.14969962288847757 rpy=0 0 0 -> xyz=0.08900000000035359 0.15400000000000424 0.22749999999999773 rpy=0 0 0
- joint Revolute88: axis -2.7155358698649516e-15 -0.9998235776537535 -0.01878333217670008 -> -2.74242071822312e-15 2.05391259555654e-14 1.000000000000006; origin xyz=-0.032900000000000734 0.1280774002974469 0.0024061448518338385 rpy=0 0 0 -> xyz=-0.03290000000000072 -3.0908609005564358e-15 -0.1281000000000023 rpy=0 0 0
- joint Revolute89: axis 0.9999999999999994 -3.0803690570051004e-15 1.7665040818381603e-14 -> 0.9999999999999992 1.8403237546193293e-14 2.7749021298199084e-15; origin xyz=0.03099999999999989 0.2063530222785827 0.036382416034325016 rpy=0 0 0 -> xyz=0.030999999999999927 0.03249999999999698 -0.20700000000000005 rpy=0 0 0
- joint Revolute90: axis 2.032489389041666e-14 0.018783332176700446 -0.9998235776537474 -> 2.100834753095154e-14 -0.9999999999999998 2.0046464488387983e-14; origin xyz=-9.71445146547012e-16 -0.06562904417471904 0.03287306740650725 rpy=0 0 0 -> xyz=-9.769962616701378e-16 0.034100000000000213 0.06499999999999914 rpy=0 0 0
- joint Revolute91: axis -1.0 3.7412631039392414e-15 -2.02925870096358e-14 -> -0.9999999999999997 -2.1042733972000734e-14 -3.3863255073556605e-15; origin xyz=0.03729999999999761 -0.0021600832003205173 0.11497971143018193 rpy=0 0 0 -> xyz=0.03729999999999738 0.11500000000000121 -1.9895196601282807e-15 rpy=0 0 0
- joint Revolute97: axis -0.999999999999997 2.143404853286814e-15 2.7487445739598234e-14 -> -0.9999999999999968 2.6758882414044968e-14 -2.6862173811482373e-15; origin xyz=0.036999999475479745 0.14377213278323475 0.0028280186039150446 rpy=0 0 0 -> xyz=0.036999999475479765 0.00012699995041472788 -0.14379988777908267 rpy=0 0 0
- joint Revolute99: axis 2.5667004481387123e-14 -0.019666798232188747 0.9998065898198966 -> 2.4983527351433608e-14 0.9999996095995696 0.0008836292804400916; origin xyz=-0.03700000000000142 0.04858072025831994 -0.02905019137945085 rpy=0 0 0 -> xyz=-0.0370000000000014 -0.029957574082523877 -0.048026490139191934 rpy=0 0 0
- joint Rigid111: origin xyz=0.05720000000000043 0.07999999999999963 -9.159339953157541e-16 rpy=0 0 0 -> xyz=0.057200000000000445 -1.5099033134902129e-15 -0.07999999999999922 rpy=0 0 0
- joint Rigid113: origin xyz=0.05720000000000827 0.07999999999999963 -2.220446049250313e-16 rpy=0 0 0 -> xyz=0.057200000000008244 6.039613253960852e-16 -0.07999999999999953 rpy=0 0 0
- joint Rigid71: origin xyz=-0.017677669529662474 0.037254823621300504 0.013057539030648296 rpy=0 0 0 -> xyz=-0.01767766952966248 0.01235546566171287 -0.03749351513093174 rpy=0 0 0
